File: pipan8l/pcb/pipan8l.kicad_pcb (KiCad board)
At the start: 2 copper layers, 262.3 x 76.2 mm, 26 parts, among them J1 2x18edgecon, J2 2x18edgecon, J3 2x18edgecon, J4 2x18edgecon, J5 Conn_02x20_Odd_Even, J6 Conn_01x02_Pin, J7 Conn_01x16, Q1 2N3904, U1 MCP23017, U2 MCP23017, U3 MCP23017, U4 MCP23017, U5 MCP23017

Commit message: rename pipanel to pipan8l and reference pdp8v github branch
Parts:
- J1, J2, J3, J4: footprint mypipanelfoots:2x18-edge -> mypipan8lfoots:2x18-edge
