File: pipan8l/pcb/pipan8l.kicad_sch (KiCad schematic)
At the start: 26 parts, among them J1 2x18edgecon, J2 2x18edgecon, J3 2x18edgecon, J4 2x18edgecon, J5 Conn_02x20_Odd_Even, J6 Conn_01x02_Pin, J7 Conn_01x16, Q1 2N3904, U1 MCP23017, U2 MCP23017, U3 MCP23017, U4 MCP23017, U5 MCP23017

Commit message: rename pipanel to pipan8l and reference pdp8v github branch
Parts:
- J1, J2, J3, J4: footprint mypipanelfoots:2x18-edge -> mypipan8lfoots:2x18-edge; symbol mypipanellib:2x18edgecon -> mypipan8llib:2x18edgecon
- U1, U2, U3, U4, U5: symbol mypipanellib:MCP23017 -> mypipan8llib:MCP23017
Changed lines of the file:
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@@
     (effects (font (size 1.27 1.27)) (justify left bottom))
   )
-  (symbol (lib_id "mypipanellib:MCP23017") (at 52.07 116.84 270) (unit 1)
+  (symbol (lib_id "mypipan8llib:MCP23017") (at 52.07 116.84 270) (unit 1)
     (in_bom yes) (on_board yes) (dnp no) (fields_autoplaced)
     (property "Reference" "U5" (at 91.44 109.9119 90)
@@
     (pin "12")
     (instances
-      (project "pipanel"
+      (project "pipan8l"
         (path "/79b05002-547f-468d-866c-9f8555f2e009"
           (reference "U5") (unit 1)
@@
     (pin "1")
     (instances
-      (project "pipanel"
+      (project "pipan8l"
         (path "/79b05002-547f-468d-866c-9f8555f2e009"
           (reference "R3") (unit 1)
@@
     )
     (instances
-      (project "pipanel"
+      (project "pipan8l"
         (path "/79b05002-547f-468d-866c-9f8555f2e009"
           (reference "H1") (unit 1)
@@
     (pin "11")
     (instances
-      (project "pipanel"
+      (project "pipan8l"
         (path "/79b05002-547f-468d-866c-9f8555f2e009"
           (reference "J7") (unit 1)
@@
     (pin "15")
     (instances
-      (project "pipanel"
+      (project "pipan8l"
         (path "/79b05002-547f-468d-866c-9f8555f2e009"
           (reference "J5") (unit 1)
@@
     )
   )
-  (symbol (lib_id "mypipanellib:2x18edgecon") (at 274.32 264.16 270) (unit 1)
+  (symbol (lib_id "mypipan8llib:2x18edgecon") (at 274.32 264.16 270) (unit 1)
     (in_bom yes) (on_board yes) (dnp no) (fields_autoplaced)
     (property "Reference" "J2" (at 273.05 267.97 90)
@@
       (effects (font (size 1.27 1.27)))
     )
-    (property "Footprint" "mypipanelfoots:2x18-edge" (at 274.32 264.16 0)
+    (property "Footprint" "mypipan8lfoots:2x18-edge" (at 274.32 264.16 0)
       (effects (font (size 1.27 1.27)) hide)
     )
@@
     (pin "B2")
     (instances
-      (project "pipanel"
+      (project "pipan8l"
         (path "/79b05002-547f-468d-866c-9f8555f2e009"
           (reference "J2") (unit 1)
@@
     )
   )
-  (symbol (lib_id "mypipanellib:2x18edgecon") (at 76.2 264.16 270) (unit 1)
+  (symbol (lib_id "mypipan8llib:2x18edgecon") (at 76.2 264.16 270) (unit 1)
     (in_bom yes) (on_board yes) (dnp no) (fields_autoplaced)
     (property "Reference" "J4" (at 74.93 267.97 90)
@@
       (effects (font (size 1.27 1.27)))
     )
-    (property "Footprint" "mypipanelfoots:2x18-edge" (at 76.2 264.16 0)
+    (property "Footprint" "mypipan8lfoots:2x18-edge" (at 76.2 264.16 0)
       (effects (font (size 1.27 1.27)) hide)
     )
@@
     (pin "B2")
     (instances
-      (project "pipanel"
+      (project "pipan8l"
         (path "/79b05002-547f-468d-866c-9f8555f2e009"
           (reference "J4") (unit 1)
@@
     (pin "1")
     (instances
-      (project "pipanel"
+      (project "pipan8l"
         (path "/79b05002-547f-468d-866c-9f8555f2e009"
           (reference "R1") (unit 1)
@@
     )
   )
-  (symbol (lib_id "mypipanellib:MCP23017") (at 260.35 116.84 270) (unit 1)
+  (symbol (lib_id "mypipan8llib:MCP23017") (at 260.35 116.84 270) (unit 1)
     (in_bom yes) (on_board yes) (dnp no) (fields_autoplaced)
     (property "Reference" "U2" (at 299.72 109.9119 90)
@@
     (pin "12")
     (instances
-      (project "pipanel"
+      (project "pipan8l"
         (path "/79b05002-547f-468d-866c-9f8555f2e009"
           (reference "U2") (unit 1)
@@
     (pin "1")
     (instances
-      (project "pipanel"
+      (project "pipan8l"
         (path "/79b05002-547f-468d-866c-9f8555f2e009"
           (reference "#PWR01") (unit 1)
@@
     (pin "1")
     (instances
-      (project "pipanel"
+      (project "pipan8l"
         (path "/79b05002-547f-468d-866c-9f8555f2e009"
           (reference "C5") (unit 1)
@@
     )
     (instances
-      (project "pipanel"
+      (project "pipan8l"
         (path "/79b05002-547f-468d-866c-9f8555f2e009"
           (reference "H2") (unit 1)
@@
     )
     (instances
-      (project "pipanel"
+      (project "pipan8l"
         (path "/79b05002-547f-468d-866c-9f8555f2e009"
           (reference "H3") (unit 1)
@@
     (pin "1")
     (instances
-      (project "pipanel"
+      (project "pipan8l"
         (path "/79b05002-547f-468d-866c-9f8555f2e009"
           (reference "#PWR03") (unit 1)
@@
     (pin "1")
     (instances
-      (project "pipanel"
+      (project "pipan8l"
         (path "/79b05002-547f-468d-866c-9f8555f2e009"
           (reference "C3") (unit 1)
@@
     (pin "2")
     (instances
-      (project "pipanel"
+      (project "pipan8l"
         (path "/79b05002-547f-468d-866c-9f8555f2e009"
           (reference "C6") (unit 1)
@@
     )
   )
-  (symbol (lib_id "mypipanellib:MCP23017") (at 121.92 116.84 270) (unit 1)
+  (symbol (lib_id "mypipan8llib:MCP23017") (at 121.92 116.84 270) (unit 1)
     (in_bom yes) (on_board yes) (dnp no) (fields_autoplaced)
     (property "Reference" "U4" (at 161.29 109.9119 90)
@@
     (pin "12")
     (instances
-      (project "pipanel"
+      (project "pipan8l"
         (path "/79b05002-547f-468d-866c-9f8555f2e009"
           (reference "U4") (unit 1)
@@
     (pin "1")
     (instances
-      (project "pipanel"
+      (project "pipan8l"
         (path "/79b05002-547f-468d-866c-9f8555f2e009"
           (reference "R2") (unit 1)
@@
     )
   )
-  (symbol (lib_id "mypipanellib:2x18edgecon") (at 373.38 264.16 270) (unit 1)
+  (symbol (lib_id "mypipan8llib:2x18edgecon") (at 373.38 264.16 270) (unit 1)
     (in_bom yes) (on_board yes) (dnp no) (fields_autoplaced)
     (property "Reference" "J1" (at 372.11 267.97 90)
@@
       (effects (font (size 1.27 1.27)))
     )
-    (property "Footprint" "mypipanelfoots:2x18-edge" (at 373.38 264.16 0)
+    (property "Footprint" "mypipan8lfoots:2x18-edge" (at 373.38 264.16 0)
       (effects (font (size 1.27 1.27)) hide)
     )
@@
     (pin "B2")
     (instances
-      (project "pipanel"
+      (project "pipan8l"
         (path "/79b05002-547f-468d-866c-9f8555f2e009"
           (reference "J1") (unit 1)
@@
     (pin "1")
     (instances
-      (project "pipanel"
+      (project "pipan8l"
         (path "/79b05002-547f-468d-866c-9f8555f2e009"
           (reference "C1") (unit 1)
@@
     (pin "2")
     (instances
-      (project "pipanel"
+      (project "pipan8l"
         (path "/79b05002-547f-468d-866c-9f8555f2e009"
           (reference "J6") (unit 1)
@@
     )
   )
-  (symbol (lib_id "mypipanellib:MCP23017") (at 334.01 118.11 270) (unit 1)
+  (symbol (lib_id "mypipan8llib:MCP23017") (at 334.01 118.11 270) (unit 1)
     (in_bom yes) (on_board yes) (dnp no) (fields_autoplaced)
     (property "Reference" "U1" (at 373.38 111.1819 90)
@@
     (pin "12")
     (instances
-      (project "pipanel"
+      (project "pipan8l"
         (path "/79b05002-547f-468d-866c-9f8555f2e009"
           (reference "U1") (unit 1)
@@
     (pin "3")
     (instances
-      (project "pipanel"
+      (project "pipan8l"
         (path "/79b05002-547f-468d-866c-9f8555f2e009"
           (reference "Q1") (unit 1)
@@
     (pin "1")
     (instances
-      (project "pipanel"
+      (project "pipan8l"
         (path "/79b05002-547f-468d-866c-9f8555f2e009"
           (reference "C2") (unit 1)
@@
     )
   )
-  (symbol (lib_id "mypipanellib:2x18edgecon") (at 175.26 264.16 270) (unit 1)
+  (symbol (lib_id "mypipan8llib:2x18edgecon") (at 175.26 264.16 270) (unit 1)
     (in_bom yes) (on_board yes) (dnp no) (fields_autoplaced)
     (property "Reference" "J3" (at 173.99 267.97 90)
@@
       (effects (font (size 1.27 1.27)))
     )
-    (property "Footprint" "mypipanelfoots:2x18-edge" (at 175.26 264.16 0)
+    (property "Footprint" "mypipan8lfoots:2x18-edge" (at 175.26 264.16 0)
       (effects (font (size 1.27 1.27)) hide)
     )
@@
     (pin "B2")
     (instances
-      (project "pipanel"
+      (project "pipan8l"
         (path "/79b05002-547f-468d-866c-9f8555f2e009"
           (reference "J3") (unit 1)
@@
     (pin "1")
     (instances
-      (project "pipanel"
+      (project "pipan8l"
         (path "/79b05002-547f-468d-866c-9f8555f2e009"
           (reference "C4") (unit 1)
@@
     )
     (instances
-      (project "pipanel"
+      (project "pipan8l"
         (path "/79b05002-547f-468d-866c-9f8555f2e009"
           (reference "H4") (unit 1)
@@
     )
   )
-  (symbol (lib_id "mypipanellib:MCP23017") (at 191.77 116.84 270) (unit 1)
+  (symbol (lib_id "mypipan8llib:MCP23017") (at 191.77 116.84 270) (unit 1)
     (in_bom yes) (on_board yes) (dnp no) (fields_autoplaced)
     (property "Reference" "U3" (at 231.14 109.9119 90)
@@
     (pin "12")
     (instances
-      (project "pipanel"
+      (project "pipan8l"
         (path "/79b05002-547f-468d-866c-9f8555f2e009"
           (reference "U3") (unit 1)
@@
     (pin "1")
     (instances
-      (project "pipanel"
+      (project "pipan8l"
         (path "/79b05002-547f-468d-866c-9f8555f2e009"
           (reference "#PWR02") (unit 1)
