File: pipan8l/pcb3/pipan8l.kicad_pcb (KiCad board)
At the start: 2 copper layers, 262.3 x 76.2 mm, 56 parts, among them J1 2x18edgecon, J2 2x18edgecon, J3 2x18edgecon, J4 2x18edgecon, J5 Conn_02x20_Odd_Even, J6 Conn_01x02_Pin, J7 Conn_01x16, J8 Conn_01x12, Q1 2N3906, Q10 2N3906, Q11 2N3906, Q12 2N3906, Q13 2N3906, Q14 2N3906, Q15 2N3906, Q16 2N3906, Q2 2N3906, Q3 2N3906, Q4 2N3906, Q5 2N3906, Q6 2N3906, Q7 2N3906, Q8 2N3906, Q9 2N3906, U1 MCP23017, U2 MCP23017, U3 MCP23017, U4 MCP23017

Commit message: add pipan8l/pcb3x and little updates for pcb3
  pcb3  - plugs into backplane for console access with console in place
  pcb3x - backplane pin straightener/insulator/spacer for use with pcb3
Parts:
- J1: footprint mypipan8lfoots:backpins -> mypipan8lfoots:backpins-A
- J2: footprint mypipan8lfoots:backpins -> mypipan8lfoots:backpins-B
- J3: footprint mypipan8lfoots:backpins -> mypipan8lfoots:backpins-C
- J4: footprint mypipan8lfoots:backpins -> mypipan8lfoots:backpins-D
- moved C6 0.22 mm to (248.9, 24.1)
- moved J8 0.07 mm to (201.9, 10.2)
- moved C2 0.06 mm to (27.9, 26.7)
- moved C3 0.06 mm to (97.8, 26.7)
- moved C4 0.06 mm to (161.3, 26.7)
- moved C5 0.06 mm to (231.8, 26.7)
Connections:
- J2 pad C2: /BC2GND -> GND
- J3 pad C2: /CC2GND -> GND
- U2 pad 21: /SR10 -> /RSR10
- U2 pad 22: /SR09 -> /RSR09
- U2 pad 23: /SR00 -> /SR10
- U2 pad 24: Net-(J8-Pin_8) -> /SR09
- U2 pad 25: Net-(J8-Pin_6) -> /SR00
- U2 pad 4: Net-(J8-Pin_7) -> Net-(J8-Pin_6)
- U2 pad 5: Net-(J8-Pin_9) -> Net-(J8-Pin_7)
- U2 pad 6: Net-(J8-Pin_10) -> Net-(J8-Pin_8)
- U2 pad 7: /RSR09 -> Net-(J8-Pin_9)
- U2 pad 8: /RSR10 -> Net-(J8-Pin_10)
Routing:
- net GND: track 546.2 -> 672.2 mm
- net /SCL: track 306.0 -> 292.8 mm
- net Net-(J8-Pin_6): track 36.6 -> 29.0 mm
- net /RSR09: track 41.8 -> 34.6 mm
- net Net-(J8-Pin_8): track 35.6 -> 29.0 mm
- net /RSR10: track 42.6 -> 37.1 mm
- net /SR00: track 89.0 -> 85.0 mm
- net /SR10: track 63.0 -> 67.0 mm
- net /SR09: track 65.6 -> 68.8 mm
- net Net-(J8-Pin_10): track 26.9 -> 29.1 mm
- net Net-(J8-Pin_9): track 26.9 -> 28.4 mm
- net VCC: track 310.0 -> 308.5 mm
- net Net-(J8-Pin_7): track 28.0 -> 29.0 mm
- net /MPRT: track 46.7 -> 46.0 mm
Other:
- board text added: "PIPAN8L 2025-01-02"
- board text removed: "PIPAN8L 2025-01-01"
