File: pipan8l/pcb3/z8lfpan.kicad_sch (KiCad schematic)
At the start: 64 parts, among them J1 2x18edgecon, J2 2x18edgecon, J3 2x18edgecon, J4 2x18edgecon, J5 Conn_02x20_Odd_Even, J6 Conn_01x02_Pin, J7 Conn_01x16, J8 Conn_01x12, Q1 2N3906, Q10 2N3906, Q11 2N3906, Q12 2N3906, Q13 2N3906, Q14 2N3906, Q15 2N3906, Q16 2N3906, Q17 2N7000, Q18 2N7000, Q2 2N3906, Q3 2N3906, Q4 2N3906, Q5 2N3906, Q6 2N3906, Q7 2N3906, Q8 2N3906, Q9 2N3906, U1 MCP23017, U2 MCP23017, U3 MCP23017, U4 MCP23017

Commit message: rename pipan8l pcb3 to z8lfpan - it is for use with zynq stuff
Parts:
- J1: footprint mypipan8lfoots:backpins-A -> myz8lfpanfoots:backpins-A; symbol mypipan8llib:2x18edgecon -> myz8lfpanlib:2x18edgecon
- J2: footprint mypipan8lfoots:backpins-B -> myz8lfpanfoots:backpins-B; symbol mypipan8llib:2x18edgecon -> myz8lfpanlib:2x18edgecon
- J3: footprint mypipan8lfoots:backpins-C -> myz8lfpanfoots:backpins-C; symbol mypipan8llib:2x18edgecon -> myz8lfpanlib:2x18edgecon
- J4: footprint mypipan8lfoots:backpins-D -> myz8lfpanfoots:backpins-D; symbol mypipan8llib:2x18edgecon -> myz8lfpanlib:2x18edgecon
- U1, U2, U3, U4: symbol mypipan8llib:MCP23017 -> myz8lfpanlib:MCP23017
