File: zturn/zturn36/zturn36.kicad_sch (KiCad schematic)
At the start: 66 parts, among them J11 Conn_02x40_Odd_Even, J12 Conn_02x40_Odd_Even, J5V1 Conn_01x03, U1 74AXP4T245, U10 74AXP4T245, U11 74AXP4T245, U12 74AXP4T245, U13 74AXP4T245, U14 LM3940_TO220, U2 74AXP4T245, U3 74AXP4T245, U4 74AXP4T245, U5 74AXP4T245, U6 74AXP4T245, U7 74AXP4T245, U8 74AXP4T245, U9 74AXP4T245

Commit message: use transistors for bus drivers instead of chips
to handle the 180 & 220-ohm pullups
Parts:
- removed C2: 10u, Capacitor_SMD:C_1206_3216Metric, symbol Device:C
- removed CA4, CA5, CA6, CA7, CB4, CB5, CB6, CB7: 0.1u, Capacitor_SMD:C_0201_0603Metric, symbol Device:C
- removed R2: 10K, Resistor_SMD:R_0201_0603Metric, symbol Device:R_US
- removed U4, U5, U6, U7: 74AXP4T245, Package_SO:TSSOP-16_4.4x5mm_P0.65mm, symbol mylibrary:74AXP4T245
- added Q1, Q2, Q3, Q4, Q5, Q6, Q7, Q8, Q9: SSM6N15AFU, Package_TO_SOT_SMD:SOT-363_SC-70-6, symbol mylibrary:SSM6N15AFU
Connections:
- net +3V3: no longer U2.3 (2A>2B), U8.2 (1A>1B)
- net DMABUSA: now also Q2.5 (G2)
- net DMABUSB: now also Q3.2 (G1)
- net DMABUSC: now also Q4.5 (G2)
- net DMABUSD: now also Q5.5 (G2)
- net DMABUSE: now also Q6.2 (G1)
- net DMABUSF: now also Q7.2 (G1)
- net DMABUSH: now also Q2.2 (G1)
- net DMABUSJ: now also Q3.5 (G2)
- net DMABUSK: now also Q4.2 (G1)
- net DMABUSL: now also Q6.5 (G2)
- net DMABUSM: now also Q7.5 (G2)
- net DMABUSN: now also Q9.2 (G1)
- net GND: now also U2.3 (2A>2B), U8.2 (1A>1B), Q1.1 (S1), Q1.4 (S2), Q2.1 (S1), Q2.4 (S2), Q3.1 (S1), Q3.4 (S2), Q4.1 (S1), Q4.4 (S2), Q5.1 (S1), Q5.4 (S2), Q6.1 (S1), Q6.4 (S2), Q7.1 (S1), Q7.4 (S2), Q8.1 (S1), Q8.4 (S2), Q9.1 (S1), Q9.4 (S2)
- net MEMBUSE: now also J12.66 (Pin_66); no longer J12.64 (Pin_64)
- net MEMBUSF: now also J12.62 (Pin_62); no longer J12.56 (Pin_56)
- net MEMBUSM: now also J12.64 (Pin_64); no longer J12.58 (Pin_58)
- net MEMBUSN: now also J12.58 (Pin_58); no longer J12.54 (Pin_54)
- net iB36V1: now also J11.63 (Pin_63), Q1.5 (G2); no longer J12.62 (Pin_62), U2.7 (2A2)
- net iCA_INCREMENT: now also J11.22 (Pin_22); no longer J11.26 (Pin_26)
- net iD36B2: now also J11.26 (Pin_26), Q8.5 (G2); no longer J11.11 (Pin_11), U8.4 (1A1)
- net iDATA_IN: now also Q8.2 (G1)
- net iMEMINCR: now also J11.18 (Pin_18), Q9.5 (G2); no longer J11.7 (Pin_7), U8.5 (1A2)
- net i_BRK_RQST: now also Q5.2 (G1)
- net i_EXTDMAADD_12: now also J11.20 (Pin_20); no longer J11.22 (Pin_22)
- net i_INT_INHIBIT: now also J11.65 (Pin_65), Q1.2 (G1); no longer J12.66 (Pin_66), U2.6 (2A1)
- net jB36V1: now also Q1.3 (D2); no longer U2.10 (2B2)
- net jD36B2: now also Q8.3 (D2); no longer U8.13 (1B1)
- net jDATA_IN: now also Q8.6 (D1)
- net jMEMINCR: now also Q9.3 (D2); no longer U8.12 (1B2)
- net j_BRK_RQST: now also Q5.6 (D1)
- net j_DMAADDR_00: now also Q2.6 (D1)
- net j_DMAADDR_01: now also Q2.3 (D2)
- net j_DMAADDR_02: now also Q4.6 (D1)
- net j_DMAADDR_03: now also Q4.3 (D2)
- net j_DMAADDR_04: now also Q6.6 (D1)
- net j_DMAADDR_05: now also Q6.3 (D2)
- net j_DMAADDR_06: now also Q7.6 (D1)
- net j_DMAADDR_07: now also Q7.3 (D2)
- net j_DMAADDR_08: now also Q9.6 (D1)
- net j_DMAADDR_09: now also Q3.3 (D2)
- net j_DMAADDR_10: now also Q3.6 (D1)
- net j_DMAADDR_11: now also Q5.3 (D2)
- net j_INT_INHIBIT: now also Q1.6 (D1); no longer U2.11 (2B1)
- net oB_BREAK: now also J11.16 (Pin_16); no longer J11.20 (Pin_20)
- net oD35B2: now also J11.7 (Pin_7); no longer J11.16 (Pin_16)
- net oJMP_JMS: now also J12.52 (Pin_52), U2.7 (2A2); no longer J11.63 (Pin_63)
- net o_ADDR_ACCEPT: now also J11.11 (Pin_11); no longer J11.18 (Pin_18)
- net o_KEY_LOAD: now also J12.56 (Pin_56), U2.6 (2A1); no longer J11.65 (Pin_65)
- net o_LOAD_SF: now also J12.48 (Pin_48); no longer J12.52 (Pin_52)
- net pJMP_JMS: now also U2.10 (2B2)
- net p_KEY_LOAD: now also U2.11 (2B1)
- net x_MEM: now also J12.54 (Pin_54); no longer J12.48 (Pin_48)
Other:
- moved on the sheet: JB36, JC36, JD36, U1, U11, U3, U9

Commit message: update net names on zturn pcbs to match active high/low signal type
Connections:
- net _rBMB renamed r_BMB
- net _rMA renamed r_MA
- net _xINPUTBUS renamed x_INPUTBUS
- net iBEMA renamed i_BEMA
- net iMEM07 renamed iMEM_07
- net iMEMINCR renamed i_MEMINCR
- net iTHREECYCLE renamed i_3CYCLE
- net i_INT_RQST renamed iINT_RQST
- net jMEMINCR renamed j_MEMINCR
- net oBWC_OVERFLOW renamed o_BWC_OVERFLOW
- net oB_BREAK renamed o_B_BREAK
- net o_BUSINIT renamed oBUSINIT
- net pB_BREAK renamed p_B_BREAK
- net p_BUSINIT renamed pBUSINIT
Changed lines of the file:
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@@
     (effects (font (size 1.27 1.27)) (justify left bottom))
   )
-  (label "p_BUSINIT" (at 430.53 233.68 0) (fields_autoplaced)
+  (label "pBUSINIT" (at 430.53 233.68 0) (fields_autoplaced)
     (effects (font (size 1.27 1.27)) (justify left bottom))
   )
@@
     (effects (font (size 1.27 1.27)) (justify left bottom))
   )
-  (label "o_BUSINIT" (at 13.97 220.98 0) (fields_autoplaced)
+  (label "oBUSINIT" (at 13.97 220.98 0) (fields_autoplaced)
     (effects (font (size 1.27 1.27)) (justify left bottom))
   )
@@
     (effects (font (size 1.27 1.27)) (justify left bottom))
   )
-  (label "oB_BREAK" (at 250.19 231.14 0) (fields_autoplaced)
+  (label "o_B_BREAK" (at 250.19 231.14 0) (fields_autoplaced)
     (effects (font (size 1.27 1.27)) (justify left bottom))
   )
@@
     (effects (font (size 1.27 1.27)) (justify left bottom))
   )
-  (label "pB_BREAK" (at 290.83 231.14 0) (fields_autoplaced)
+  (label "p_B_BREAK" (at 290.83 231.14 0) (fields_autoplaced)
     (effects (font (size 1.27 1.27)) (justify left bottom))
   )
@@
     (effects (font (size 1.27 1.27)) (justify left bottom))
   )
-  (label "iMEM07" (at 13.97 264.16 0) (fields_autoplaced)
+  (label "iMEM_07" (at 13.97 264.16 0) (fields_autoplaced)
     (effects (font (size 1.27 1.27)) (justify left bottom))
   )
@@
     (effects (font (size 1.27 1.27)) (justify left bottom))
   )
-  (label "iMEM07" (at 209.55 124.46 0) (fields_autoplaced)
+  (label "iMEM_07" (at 209.55 124.46 0) (fields_autoplaced)
     (effects (font (size 1.27 1.27)) (justify left bottom))
   )
@@
     (effects (font (size 1.27 1.27)) (justify left bottom))
   )
-  (label "oB_BREAK" (at 54.61 223.52 0) (fields_autoplaced)
+  (label "o_B_BREAK" (at 54.61 223.52 0) (fields_autoplaced)
     (effects (font (size 1.27 1.27)) (justify left bottom))
   )
@@
     (effects (font (size 1.27 1.27)) (justify left bottom))
   )
-  (label "iTHREECYCLE" (at 208.28 191.77 0) (fields_autoplaced)
+  (label "i_3CYCLE" (at 208.28 191.77 0) (fields_autoplaced)
     (effects (font (size 1.27 1.27)) (justify left bottom))
   )
@@
     (effects (font (size 1.27 1.27)) (justify left bottom))
   )
-  (label "pB_BREAK" (at 430.53 208.28 0) (fields_autoplaced)
+  (label "p_B_BREAK" (at 430.53 208.28 0) (fields_autoplaced)
     (effects (font (size 1.27 1.27)) (justify left bottom))
   )
@@
     (effects (font (size 1.27 1.27)) (justify left bottom))
   )
-  (label "oBWC_OVERFLOW" (at 171.45 207.01 0) (fields_autoplaced)
+  (label "o_BWC_OVERFLOW" (at 171.45 207.01 0) (fields_autoplaced)
     (effects (font (size 1.27 1.27)) (justify left bottom))
   )
@@
     (effects (font (size 1.27 1.27)) (justify left bottom))
   )
-  (label "_xINPUTBUS" (at 171.45 266.7 0) (fields_autoplaced)
+  (label "x_INPUTBUS" (at 171.45 266.7 0) (fields_autoplaced)
     (effects (font (size 1.27 1.27)) (justify left bottom))
   )
@@
     (effects (font (size 1.27 1.27)) (justify left bottom))
   )
-  (label "jMEMINCR" (at 430.53 223.52 0) (fields_autoplaced)
+  (label "j_MEMINCR" (at 430.53 223.52 0) (fields_autoplaced)
     (effects (font (size 1.27 1.27)) (justify left bottom))
   )
@@
     (effects (font (size 1.27 1.27)) (justify left bottom))
   )
-  (label "i_INT_RQST" (at 208.28 279.4 0) (fields_autoplaced)
+  (label "iINT_RQST" (at 208.28 279.4 0) (fields_autoplaced)
     (effects (font (size 1.27 1.27)) (justify left bottom))
   )
@@
     (effects (font (size 1.27 1.27)) (justify left bottom))
   )
-  (label "jMEMINCR" (at 307.34 172.72 0) (fields_autoplaced)
+  (label "j_MEMINCR" (at 307.34 172.72 0) (fields_autoplaced)
     (effects (font (size 1.27 1.27)) (justify left bottom))
   )
@@
     (effects (font (size 1.27 1.27)) (justify left bottom))
   )
-  (label "i_INT_RQST" (at 82.55 241.3 0) (fields_autoplaced)
+  (label "iINT_RQST" (at 82.55 241.3 0) (fields_autoplaced)
     (effects (font (size 1.27 1.27)) (justify left bottom))
   )
@@
     (effects (font (size 1.27 1.27)) (justify left bottom))
   )
-  (label "iTHREECYCLE" (at 54.61 243.84 0) (fields_autoplaced)
+  (label "i_3CYCLE" (at 54.61 243.84 0) (fields_autoplaced)
     (effects (font (size 1.27 1.27)) (justify left bottom))
   )
@@
     (effects (font (size 1.27 1.27)) (justify left bottom))
   )
-  (label "_rMA" (at 209.55 119.38 0) (fields_autoplaced)
+  (label "r_MA" (at 209.55 119.38 0) (fields_autoplaced)
     (effects (font (size 1.27 1.27)) (justify left bottom))
   )
@@
     (effects (font (size 1.27 1.27)) (justify left bottom))
   )
-  (label "iBEMA" (at 13.97 261.62 0) (fields_autoplaced)
+  (label "i_BEMA" (at 13.97 261.62 0) (fields_autoplaced)
     (effects (font (size 1.27 1.27)) (justify left bottom))
   )
@@
     (effects (font (size 1.27 1.27)) (justify left bottom))
   )
-  (label "o_BUSINIT" (at 361.95 284.48 0) (fields_autoplaced)
+  (label "oBUSINIT" (at 361.95 284.48 0) (fields_autoplaced)
     (effects (font (size 1.27 1.27)) (justify left bottom))
   )
@@
     (effects (font (size 1.27 1.27)) (justify left bottom))
   )
-  (label "oBWC_OVERFLOW" (at 13.97 215.9 0) (fields_autoplaced)
+  (label "o_BWC_OVERFLOW" (at 13.97 215.9 0) (fields_autoplaced)
     (effects (font (size 1.27 1.27)) (justify left bottom))
   )
@@
     (effects (font (size 1.27 1.27)) (justify left bottom))
   )
-  (label "_xINPUTBUS" (at 123.19 238.76 0) (fields_autoplaced)
+  (label "x_INPUTBUS" (at 123.19 238.76 0) (fields_autoplaced)
     (effects (font (size 1.27 1.27)) (justify left bottom))
   )
@@
     (effects (font (size 1.27 1.27)) (justify left bottom))
   )
-  (label "p_BUSINIT" (at 402.59 284.48 0) (fields_autoplaced)
+  (label "pBUSINIT" (at 402.59 284.48 0) (fields_autoplaced)
     (effects (font (size 1.27 1.27)) (justify left bottom))
   )
@@
     (effects (font (size 1.27 1.27)) (justify left bottom))
   )
-  (label "_rMA" (at 13.97 259.08 0) (fields_autoplaced)
+  (label "r_MA" (at 13.97 259.08 0) (fields_autoplaced)
     (effects (font (size 1.27 1.27)) (justify left bottom))
   )
@@
     (effects (font (size 1.27 1.27)) (justify left bottom))
   )
-  (label "iMEMINCR" (at 54.61 226.06 0) (fields_autoplaced)
+  (label "i_MEMINCR" (at 54.61 226.06 0) (fields_autoplaced)
     (effects (font (size 1.27 1.27)) (justify left bottom))
   )
@@
     (effects (font (size 1.27 1.27)) (justify left bottom))
   )
-  (label "_rBMB" (at 82.55 236.22 0) (fields_autoplaced)
+  (label "r_BMB" (at 82.55 236.22 0) (fields_autoplaced)
     (effects (font (size 1.27 1.27)) (justify left bottom))
   )
@@
     (effects (font (size 1.27 1.27)) (justify left bottom))
   )
-  (label "_rBMB" (at 171.45 276.86 0) (fields_autoplaced)
+  (label "r_BMB" (at 171.45 276.86 0) (fields_autoplaced)
     (effects (font (size 1.27 1.27)) (justify left bottom))
   )
@@
     (effects (font (size 1.27 1.27)) (justify left bottom))
   )
-  (label "iBEMA" (at 172.72 124.46 0) (fields_autoplaced)
+  (label "i_BEMA" (at 172.72 124.46 0) (fields_autoplaced)
     (effects (font (size 1.27 1.27)) (justify left bottom))
   )
@@
     (effects (font (size 1.27 1.27)) (justify left bottom))
   )
-  (label "iMEMINCR" (at 274.32 180.34 0) (fields_autoplaced)
-    (effects (font (size 1.27 1.27)) (justify left bottom))
-  )
+  (label "i_MEMINCR" (at 274.32 180.34 0) (fields_autoplaced)
+    (effects (font (size 1.27 1.27)) (justify left bottom))
+  )

Commit message: update software and further updates to firmware/pcbs
...for invertering transistors

./z8lsimtest works
Connections:
- net iB36V1 renamed i_B36V1
- net iCA_INCREMENT renamed i_CA_INCRMNT
- net iD36B2 renamed i_D36B2
- net iDATA_IN renamed i_DATA_IN
- net iMEM_07 renamed i_MEM_07
- net i_3CYCLE renamed i3CYCLE
- net i_AC_CLEAR renamed iAC_CLEAR
- net i_BEMA renamed iBEMA
- net i_BRK_RQST renamed iBRK_RQST
- net i_EMA renamed iEMA
- net i_EXTDMAADD_12 renamed iEXTDMAADD_12
- net i_INT_INHIBIT renamed iINT_INHIBIT
- net i_IO_SKIP renamed iIO_SKIP
- net i_MEMINCR renamed iMEMINCR
- net o_B_RUN renamed oB_RUN
Changed lines of the file:
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@@
     (effects (font (size 1.27 1.27)) (justify left bottom))
   )
-  (label "o_B_RUN" (at 208.28 284.48 0) (fields_autoplaced)
+  (label "oB_RUN" (at 208.28 284.48 0) (fields_autoplaced)
     (effects (font (size 1.27 1.27)) (justify left bottom))
   )
@@
     (effects (font (size 1.27 1.27)) (justify left bottom))
   )
-  (label "i_INT_INHIBIT" (at 13.97 287.02 0) (fields_autoplaced)
+  (label "iINT_INHIBIT" (at 13.97 287.02 0) (fields_autoplaced)
     (effects (font (size 1.27 1.27)) (justify left bottom))
   )
@@
     (effects (font (size 1.27 1.27)) (justify left bottom))
   )
-  (label "iMEM_07" (at 13.97 264.16 0) (fields_autoplaced)
+  (label "i_MEM_07" (at 13.97 264.16 0) (fields_autoplaced)
     (effects (font (size 1.27 1.27)) (justify left bottom))
   )
@@
     (effects (font (size 1.27 1.27)) (justify left bottom))
   )
-  (label "i_IO_SKIP" (at 208.28 276.86 0) (fields_autoplaced)
+  (label "iIO_SKIP" (at 208.28 276.86 0) (fields_autoplaced)
     (effects (font (size 1.27 1.27)) (justify left bottom))
   )
@@
     (effects (font (size 1.27 1.27)) (justify left bottom))
   )
-  (label "iMEM_07" (at 209.55 124.46 0) (fields_autoplaced)
+  (label "i_MEM_07" (at 209.55 124.46 0) (fields_autoplaced)
     (effects (font (size 1.27 1.27)) (justify left bottom))
   )
@@
     (effects (font (size 1.27 1.27)) (justify left bottom))
   )
-  (label "iB36V1" (at 375.92 162.56 0) (fields_autoplaced)
+  (label "i_B36V1" (at 375.92 162.56 0) (fields_autoplaced)
     (effects (font (size 1.27 1.27)) (justify left bottom))
   )
@@
     (effects (font (size 1.27 1.27)) (justify left bottom))
   )
-  (label "i_3CYCLE" (at 208.28 191.77 0) (fields_autoplaced)
-    (effects (font (size 1.27 1.27)) (justify left bottom))
-  )
-  (label "i_INT_INHIBIT" (at 375.92 144.78 0) (fields_autoplaced)
-    (effects (font (size 1.27 1.27)) (justify left bottom))
-  )
-  (label "o_B_RUN" (at 82.55 251.46 0) (fields_autoplaced)
+  (label "i3CYCLE" (at 208.28 191.77 0) (fields_autoplaced)
+    (effects (font (size 1.27 1.27)) (justify left bottom))
+  )
+  (label "iINT_INHIBIT" (at 375.92 144.78 0) (fields_autoplaced)
+    (effects (font (size 1.27 1.27)) (justify left bottom))
+  )
+  (label "oB_RUN" (at 82.55 251.46 0) (fields_autoplaced)
     (effects (font (size 1.27 1.27)) (justify left bottom))
   )
@@
     (effects (font (size 1.27 1.27)) (justify left bottom))
   )
-  (label "i_EMA" (at 13.97 269.24 0) (fields_autoplaced)
+  (label "iEMA" (at 13.97 269.24 0) (fields_autoplaced)
     (effects (font (size 1.27 1.27)) (justify left bottom))
   )
@@
     (effects (font (size 1.27 1.27)) (justify left bottom))
   )
-  (label "i_AC_CLEAR" (at 171.45 281.94 0) (fields_autoplaced)
+  (label "iAC_CLEAR" (at 171.45 281.94 0) (fields_autoplaced)
     (effects (font (size 1.27 1.27)) (justify left bottom))
   )
@@
     (effects (font (size 1.27 1.27)) (justify left bottom))
   )
-  (label "iDATA_IN" (at 274.32 127 0) (fields_autoplaced)
+  (label "i_DATA_IN" (at 274.32 127 0) (fields_autoplaced)
     (effects (font (size 1.27 1.27)) (justify left bottom))
   )
@@
     (effects (font (size 1.27 1.27)) (justify left bottom))
   )
-  (label "i_3CYCLE" (at 54.61 243.84 0) (fields_autoplaced)
+  (label "i3CYCLE" (at 54.61 243.84 0) (fields_autoplaced)
     (effects (font (size 1.27 1.27)) (justify left bottom))
   )
@@
     (effects (font (size 1.27 1.27)) (justify left bottom))
   )
-  (label "i_BRK_RQST" (at 327.66 180.34 0) (fields_autoplaced)
+  (label "iBRK_RQST" (at 327.66 180.34 0) (fields_autoplaced)
     (effects (font (size 1.27 1.27)) (justify left bottom))
   )
@@
     (effects (font (size 1.27 1.27)) (justify left bottom))
   )
-  (label "i_BEMA" (at 13.97 261.62 0) (fields_autoplaced)
+  (label "iBEMA" (at 13.97 261.62 0) (fields_autoplaced)
     (effects (font (size 1.27 1.27)) (justify left bottom))
   )
@@
     (effects (font (size 1.27 1.27)) (justify left bottom))
   )
-  (label "iB36V1" (at 13.97 284.48 0) (fields_autoplaced)
+  (label "i_B36V1" (at 13.97 284.48 0) (fields_autoplaced)
     (effects (font (size 1.27 1.27)) (justify left bottom))
   )
@@
     (effects (font (size 1.27 1.27)) (justify left bottom))
   )
-  (label "i_EXTDMAADD_12" (at 54.61 228.6 0) (fields_autoplaced)
+  (label "iEXTDMAADD_12" (at 54.61 228.6 0) (fields_autoplaced)
     (effects (font (size 1.27 1.27)) (justify left bottom))
   )
@@
     (effects (font (size 1.27 1.27)) (justify left bottom))
   )
-  (label "iD36B2" (at 274.32 144.78 0) (fields_autoplaced)
+  (label "i_D36B2" (at 274.32 144.78 0) (fields_autoplaced)
     (effects (font (size 1.27 1.27)) (justify left bottom))
   )
@@
     (effects (font (size 1.27 1.27)) (justify left bottom))
   )
-  (label "iDATA_IN" (at 54.61 238.76 0) (fields_autoplaced)
+  (label "i_DATA_IN" (at 54.61 238.76 0) (fields_autoplaced)
     (effects (font (size 1.27 1.27)) (justify left bottom))
   )
@@
     (effects (font (size 1.27 1.27)) (justify left bottom))
   )
-  (label "iD36B2" (at 54.61 236.22 0) (fields_autoplaced)
+  (label "i_D36B2" (at 54.61 236.22 0) (fields_autoplaced)
     (effects (font (size 1.27 1.27)) (justify left bottom))
   )
@@
     (effects (font (size 1.27 1.27)) (justify left bottom))
   )
-  (label "i_MEMINCR" (at 54.61 226.06 0) (fields_autoplaced)
+  (label "iMEMINCR" (at 54.61 226.06 0) (fields_autoplaced)
     (effects (font (size 1.27 1.27)) (justify left bottom))
   )
@@
     (effects (font (size 1.27 1.27)) (justify left bottom))
   )
-  (label "i_IO_SKIP" (at 123.19 231.14 0) (fields_autoplaced)
+  (label "iIO_SKIP" (at 123.19 231.14 0) (fields_autoplaced)
     (effects (font (size 1.27 1.27)) (justify left bottom))
   )
@@
     (effects (font (size 1.27 1.27)) (justify left bottom))
   )
-  (label "i_EMA" (at 172.72 129.54 0) (fields_autoplaced)
+  (label "iEMA" (at 172.72 129.54 0) (fields_autoplaced)
     (effects (font (size 1.27 1.27)) (justify left bottom))
   )
@@
     (effects (font (size 1.27 1.27)) (justify left bottom))
   )
-  (label "i_BRK_RQST" (at 54.61 241.3 0) (fields_autoplaced)
+  (label "iBRK_RQST" (at 54.61 241.3 0) (fields_autoplaced)
     (effects (font (size 1.27 1.27)) (justify left bottom))
   )
@@
     (effects (font (size 1.27 1.27)) (justify left bottom))
   )
-  (label "iCA_INCREMENT" (at 171.45 196.85 0) (fields_autoplaced)
+  (label "i_CA_INCRMNT" (at 171.45 196.85 0) (fields_autoplaced)
     (effects (font (size 1.27 1.27)) (justify left bottom))
   )
@@
     (effects (font (size 1.27 1.27)) (justify left bottom))
   )
-  (label "i_AC_CLEAR" (at 82.55 248.92 0) (fields_autoplaced)
+  (label "iAC_CLEAR" (at 82.55 248.92 0) (fields_autoplaced)
     (effects (font (size 1.27 1.27)) (justify left bottom))
   )
@@
     (effects (font (size 1.27 1.27)) (justify left bottom))
   )
-  (label "iCA_INCREMENT" (at 54.61 231.14 0) (fields_autoplaced)
+  (label "i_CA_INCRMNT" (at 54.61 231.14 0) (fields_autoplaced)
     (effects (font (size 1.27 1.27)) (justify left bottom))
   )
@@
     (effects (font (size 1.27 1.27)) (justify left bottom))
   )
-  (label "i_BEMA" (at 172.72 124.46 0) (fields_autoplaced)
+  (label "iBEMA" (at 172.72 124.46 0) (fields_autoplaced)
     (effects (font (size 1.27 1.27)) (justify left bottom))
   )
@@
     (effects (font (size 1.27 1.27)) (justify left bottom))
   )
-  (label "i_MEMINCR" (at 274.32 180.34 0) (fields_autoplaced)
+  (label "iMEMINCR" (at 274.32 180.34 0) (fields_autoplaced)
     (effects (font (size 1.27 1.27)) (justify left bottom))
   )
@@
     (effects (font (size 1.27 1.27)) (justify left bottom))
   )
-  (label "i_EXTDMAADD_12" (at 208.28 196.85 0) (fields_autoplaced)
-    (effects (font (size 1.27 1.27)) (justify left bottom))
-  )
+  (label "iEXTDMAADD_12" (at 208.28 196.85 0) (fields_autoplaced)
+    (effects (font (size 1.27 1.27)) (justify left bottom))
+  )
