File: zturn/zturn36/zturn36.kicad_sch (KiCad schematic)
At the start: 63 parts, among them J11 Conn_02x40_Odd_Even, J12 Conn_02x40_Odd_Even, J5V1 Conn_01x03, Q1 SSM6N15AFU, Q2 SSM6N15AFU, Q3 SSM6N15AFU, Q4 SSM6N15AFU, Q5 SSM6N15AFU, Q6 SSM6N15AFU, Q7 SSM6N15AFU, Q8 SSM6N15AFU, Q9 SSM6N15AFU, U1 74AXP4T245, U10 74AXP4T245, U11 74AXP4T245, U12 74AXP4T245, U13 74AXP4T245, U2 74AXP4T245, U3 74AXP4T245, U8 74AXP4T245, U9 74AXP4T245

Commit message: put 2024-12-30 version of zturn35,36 boards back
the 2024-12-30 design had 5V I2C bus via 74AXP245s
the newer boards had 3.3V I2C bus directly on FPGA

the old boards work perfectly fine so go back to them
...rather than make new boards
Parts:
- removed R5: 2.2K, Resistor_THT:R_Axial_DIN0204_L3.6mm_D1.6mm_P5.08mm_Horizontal, symbol Device:R_US
- R4: value 2.2K -> 1K
Connections:
- net +3V3: no longer R4.1
- net +5V: now also R4.1
- net FPI2CCLK: now also U8.6 (2A1); no longer JI2C1.3 (Pin_3), R4.2
- net EPI2CDAT: now reaches JD35.22 (Pin_22)
- net EPI2CDAT: now also JI2C1.1 (Pin_1)
- net FPI2CDENA: now reaches JD35.25 (Pin_25)
- net FPI2CDENA: now also J12.25 (Pin_25)
- net EPI2CCLK: now reaches U8.11 (2B1)
- net EPI2CCLK: now also JC36.N2, JI2C1.3 (Pin_3), R4.2
- net FPI2CDDIR: now reaches JC35.35 (Pin_35)
- net FPI2CDDIR: now also J11.13 (Pin_13)
- net FPI2CDATA: now reaches JC35.36 (Pin_36)
- net FPI2CDATA: now also J11.17 (Pin_17)
- removed net FPI2CDAT: J11.17 (Pin_17), JI2C1.1 (Pin_1)
- net iMEMINCR renamed i_MEMINCR
Other:
- moved on the sheet: R4
